File: hardware/Asistente.kicad_sch (KiCad schematic)
At the start: 24 parts, among them J1 Conn_01x01_Pin, J10 Conn_01x01_Pin, J11 Conn_01x01_Pin, J12 Conn_01x01_Pin, J2 Conn_01x01_Pin, J3 Conn_01x01_Pin, J4 Conn_01x01_Pin, J5 Conn_01x01_Pin, J6 Conn_01x01_Pin, J7 Conn_01x01_Pin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

Commit message: Refactor and remove obsolete files
Parts:
- C2, C3: footprint Capacitor_SMD:C_0805_2012Metric -> Capacitor_THT:C_Disc_D5.0mm_W2.5mm_P5.00mm
- R3, R4: footprint Resistor_SMD:R_0603_1608Metric -> Resistor_THT:R_Axial_DIN0207_L6.3mm_D2.5mm_P10.16mm_Horizontal
Changed lines of the file:
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@@
 			)
 		)
-		(property "Footprint" "Resistor_SMD:R_0603_1608Metric"
+		(property "Footprint" "Resistor_THT:R_Axial_DIN0207_L6.3mm_D2.5mm_P10.16mm_Horizontal"
 			(at 103.378 82.55 90)
 			(effects
@@
 		)
 		(instances
-			(project ""
+			(project "Asistente"
 				(path "/97dc264d-c8ec-4099-a14f-39f91d52d718"
 					(reference "J1")
@@
 		)
 		(instances
-			(project ""
+			(project "Asistente"
 				(path "/97dc264d-c8ec-4099-a14f-39f91d52d718"
 					(reference "LS2")
@@
 		)
 		(instances
-			(project ""
+			(project "Asistente"
 				(path "/97dc264d-c8ec-4099-a14f-39f91d52d718"
 					(reference "J2")
@@
 		)
 		(instances
-			(project ""
+			(project "Asistente"
 				(path "/97dc264d-c8ec-4099-a14f-39f91d52d718"
 					(reference "GNDMIC1")
@@
 			)
 		)
-		(property "Footprint" "Capacitor_SMD:C_0805_2012Metric"
+		(property "Footprint" "Capacitor_THT:C_Disc_D5.0mm_W2.5mm_P5.00mm"
 			(at 96.52 72.39 0)
 			(effects
@@
 		)
 		(instances
-			(project ""
+			(project "Asistente"
 				(path "/97dc264d-c8ec-4099-a14f-39f91d52d718"
 					(reference "C3")
@@
 			)
 		)
-		(property "Footprint" "Resistor_SMD:R_0603_1608Metric"
+		(property "Footprint" "Resistor_THT:R_Axial_DIN0207_L6.3mm_D2.5mm_P10.16mm_Horizontal"
 			(at 98.298 82.55 90)
 			(effects
@@
 		)
 		(instances
-			(project ""
+			(project "Asistente"
 				(path "/97dc264d-c8ec-4099-a14f-39f91d52d718"
 					(reference "J3")
@@
 		)
 		(instances
-			(project ""
+			(project "Asistente"
 				(path "/97dc264d-c8ec-4099-a14f-39f91d52d718"
 					(reference "C1")
@@
 		)
 		(instances
-			(project ""
+			(project "Asistente"
 				(path "/97dc264d-c8ec-4099-a14f-39f91d52d718"
 					(reference "U2")
@@
 			)
 		)
-		(property "Footprint" "Capacitor_SMD:C_0805_2012Metric"
+		(property "Footprint" "Capacitor_THT:C_Disc_D5.0mm_W2.5mm_P5.00mm"
 			(at 101.6 72.39 0)
 			(effects
@@
 		)
 		(instances
-			(project ""
+			(project "Asistente"
 				(path "/97dc264d-c8ec-4099-a14f-39f91d52d718"
 					(reference "C2")
@@
 		)
 		(instances
-			(project ""
+			(project "Asistente"
 				(path "/97dc264d-c8ec-4099-a14f-39f91d52d718"
 					(reference "LS1")
@@
 		)
 		(instances
-			(project ""
+			(project "Asistente"
 				(path "/97dc264d-c8ec-4099-a14f-39f91d52d718"
 					(reference "DS1")
@@
 		)
 		(instances
-			(project ""
+			(project "Asistente"
 				(path "/97dc264d-c8ec-4099-a14f-39f91d52d718"
 					(reference "#PWR02")
@@
 		)
 		(instances
-			(project ""
+			(project "Asistente"
 				(path "/97dc264d-c8ec-4099-a14f-39f91d52d718"
 					(reference "U1")
@@
 		)
 		(instances
-			(project ""
+			(project "Asistente"
 				(path "/97dc264d-c8ec-4099-a14f-39f91d52d718"
 					(reference "J4")
@@
 		)
 		(instances
-			(project ""
+			(project "Asistente"
 				(path "/97dc264d-c8ec-4099-a14f-39f91d52d718"
 					(reference "#PWR01")
@@
 		)
 		(instances
-			(project ""
+			(project "Asistente"
 				(path "/97dc264d-c8ec-4099-a14f-39f91d52d718"
 					(reference "INMP441")
